File: kicad/V1.01 REV.B/PCB/MiniCamel_V1.01.kicad_sch (KiCad schematic)
At the start: 240 parts, among them J1 J_USB_C, J10 AUDIO_IN, J11 ESP8266 MODULE, J12 PI_ZERO_2, J13 MICRO_SD, J14 I2C_OLED, J15 USB_2, J16 I2C_EXT, J17 Wuerth Elektronik 7499010211A, J2 USB_HID, J3 USB_1, J5 J_TOSLINK_ZGY133T10, J6 AUDIO_OUT, J7 MINI_PCIE, J8 P_DE9M, J9 Conn_01x06, P1 SOM-128-EX, P2 FAN1, P3 P_CONN_01X03, Q1 Q_PMOS_GDS, Q4 NPN, SW1 PWR/RST, SW2 SYNTH, SW5 HID_PRG, U1 U_MAX16054, U10 EMC2301, U11 PCM5102A, U12 U_MIC5219-3.3YM5, U13 U_MIC5219-3.3YM5, U14 CS4237B-KQ, U15 OPA1656, U16 YAC512, U17 TL074, U18 OPA1656, U2 U_AMS1117-3.3, U4 MC74HC1G04, U5 U_MAX3243, U6 U_74LVC1G126, U7 YMF262, U8 U_74LVC1G04, U9 CH559, X2 16.9344MHz, Y1 Crystal_GND24

Commit message: 250605-01
updated revision numbers on schematic
Parts:
- JP6: now left out of the parts list
Other:
- note added: "MiniCamel 1.01 REV.C"
- note removed: "MiniCamel v1.01"
- moved on the sheet: JP6
Changed lines of the file:
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@@
 	(title_block
 		(title "MiniCamel")
-		(date "2024-06-18")
-		(rev "0.1")
+		(date "2025-06-05")
+		(rev "1.01C")
 		(company "Matt Schultz")
 		(comment 1 "Based on TinyLlama 2 by Eivind Bøhler")
@@
 		)
 	)
-	(text "MiniCamel v1.01\n"
+	(text "MiniCamel 1.01 REV.C"
 		(exclude_from_sim no)
 		(at 17.78 29.464 0)
@@
 	(symbol
 		(lib_id "Jumper:Jumper_2_Bridged")
-		(at 683.26 83.82 180)
+		(at 683.26 83.82 0)
+		(mirror y)
 		(unit 1)
-		(exclude_from_sim yes)
-		(in_bom yes)
+		(exclude_from_sim no)
+		(in_bom no)
 		(on_board yes)
 		(dnp no)
 		(property "Reference" "JP6"
-			(at 683.26 81.534 0)
+			(at 683.26 81.026 0)
 			(effects
 				(font
@@
 		)
 		(property "Value" "ESP_POWER"
-			(at 683.26 86.614 0)
+			(at 683.26 86.36 0)
 			(effects
 				(font
